Commit message: removed underscore for name arg
messed up the prefix arg in ur10wab xacro files

File: realsense2_description/urdf/_l515.urdf.xacro (robot description, xacro)
@@ -46,16 +46,16 @@
     <xacro:property name="l515_cam_color_to_imu_rz" value="0.016301375"/>
     <!-- camera body, with origin at bottom screw mount -->
-    <joint name="${name}_joint" type="fixed">
+    <joint name="${name}joint" type="fixed">
       <xacro:insert_block name="origin" />
       <parent link="${parent}"/>
-      <child link="${name}_bottom_screw_frame" />
+      <child link="${name}bottom_screw_frame" />
     </joint>
-    <link name="${name}_bottom_screw_frame"/>
-    <joint name="${name}_link_joint" type="fixed">
+    <link name="${name}bottom_screw_frame"/>
+    <joint name="${name}link_joint" type="fixed">
       <origin xyz="${l515_cam_depth_px} ${l515_cam_depth_py} ${l515_cam_depth_pz}" rpy="0 0 0"/>
-      <parent link="${name}_bottom_screw_frame"/>
-      <child link="${name}_link" />
+      <parent link="${name}bottom_screw_frame"/>
+      <child link="${name}link" />
     </joint>
-    <link name="${name}_link">
+    <link name="${name}link">
       <visual>
         <!-- the mesh origin is in the middle of the front plate -->
@@ -88,85 +88,85 @@
       </inertial>
     </link>
-    <joint name="${name}_lower_mount_joint" type="fixed">
+    <joint name="${name}lower_mount_joint" type="fixed">
       <origin xyz="${l515_cam_mount_from_glass_offset-l515_cam_depth} 0 ${l515_cam_center-abs_mount_from_center}" rpy="0 0 0" />
-      <parent link="${name}_bottom_screw_frame" />
-      <child link="${name}_lower_mount" />
+      <parent link="${name}bottom_screw_frame" />
+      <child link="${name}lower_mount" />
     </joint>
-    <link name="${name}_lower_mount"/>
-    <joint name="${name}_upper_mount_joint" type="fixed">
+    <link name="${name}lower_mount"/>
+    <joint name="${name}upper_mount_joint" type="fixed">
       <origin xyz="${l515_cam_mount_from_glass_offset-l515_cam_depth} 0 ${l515_cam_center+abs_mount_from_center}" rpy="0 0 0" />
-      <parent link="${name}_bottom_screw_frame" />
-      <child link="${name}_upper_mount" />
+      <parent link="${name}bottom_screw_frame" />
+      <child link="${name}upper_mount" />
     </joint>
-    <link name="${name}_upper_mount"/>
+    <link name="${name}upper_mount"/>
     <!-- Use the nominal extrinsics between camera frames if the calibrated extrinsics aren't being published. e.g. running the device in simulation  -->
     <xacro:if value="${use_nominal_extrinsics}">
       <!-- camera depth joints and links -->
-      <joint name="${name}_depth_joint" type="fixed">
+      <joint name="${name}depth_joint" type="fixed">
         <origin xyz="0 0 0" rpy="0 0 0"/>
-        <parent link="${name}_link"/>
-        <child link="${name}_depth_frame" />
+        <parent link="${name}link"/>
+        <child link="${name}depth_frame" />
       </joint>
-      <link name="${name}_depth_frame"/>
-      <joint name="${name}_depth_optical_joint" type="fixed">
+      <link name="${name}depth_frame"/>
+      <joint name="${name}depth_optical_joint" type="fixed">
         <origin xyz="0 0 0" rpy="${-M_PI/2} 0 ${-M_PI/2}" />
-        <parent link="${name}_depth_frame" />
-        <child link="${name}_depth_optical_frame" />
+        <parent link="${name}depth_frame" />
+        <child link="${name}depth_optical_frame" />
       </joint>
-      <link name="${name}_depth_optical_frame"/>
+      <link name="${name}depth_optical_frame"/>
       <!-- camera left IR joints and links -->
-      <joint name="${name}_infra_joint" type="fixed">
+      <joint name="${name}infra_joint" type="fixed">
         <origin xyz="0 ${l515_cam_depth_to_infra_offset} 0" rpy="0 0 0" />
-        <parent link="${name}_link" />
-        <child link="${name}_infra_frame" />
+        <parent link="${name}link" />
+        <child link="${name}infra_frame" />
       </joint>
-      <link name="${name}_infra_frame"/>
-      <joint name="${name}_infra_optical_joint" type="fixed">
+      <link name="${name}infra_frame"/>
+      <joint name="${name}infra_optical_joint" type="fixed">
         <origin xyz="0 0 0" rpy="${-M_PI/2} 0 ${-M_PI/2}" />
-        <parent link="${name}_infra_frame" />
-        <child link="${name}_infra_optical_frame" />
+        <parent link="${name}infra_frame" />
+        <child link="${name}infra_optical_frame" />
       </joint>
-      <link name="${name}_infra_optical_frame"/>
+      <link name="${name}infra_optical_frame"/>
       <!-- camera color joints and links -->
-      <joint name="${name}_color_joint" type="fixed">
+      <joint name="${name}color_joint" type="fixed">
         <origin xyz="0 0 ${-l515_cam_transmitter_to_depth_pz+l515_cam_transmitter_to_color_pz}" rpy="0 0 0" />
-        <parent link="${name}_link" />
-        <child link="${name}_color_frame" />
+        <parent link="${name}link" />
+        <child link="${name}color_frame" />
       </joint>
-      <link name="${name}_color_frame"/>
-      <joint name="${name}_color_optical_joint" type="fixed">
+      <link name="${name}color_frame"/>
+      <joint name="${name}color_optical_joint" type="fixed">
         <origin xyz="0 0 0" rpy="${-M_PI/2} 0 ${-M_PI/2}" />
-        <parent link="${name}_color_frame" />
-        <child link="${name}_color_optical_frame" />
+        <parent link="${name}color_frame" />
+        <child link="${name}color_optical_frame" />
       </joint>
-      <link name="${name}_color_optical_frame"/>
+      <link name="${name}color_optical_frame"/>
       <!-- camera IMU joints and links -->
-      <link name="${name}_gyro_frame" />
-      <link name="${name}_gyro_optical_frame" />
-      <link name="${name}_accel_frame" />
-      <link name="${name}_accel_optical_frame" />
-      <joint name="${name}_gyro_joint" type="fixed">
+      <link name="${name}gyro_frame" />
+      <link name="${name}gyro_optical_frame" />
+      <link name="${name}accel_frame" />
+      <link name="${name}accel_optical_frame" />
+      <joint name="${name}gyro_joint" type="fixed">
         <origin xyz = "${l515_cam_color_to_imu_px} ${l515_cam_color_to_imu_py} ${l515_cam_color_to_imu_pz}" rpy = "${l515_cam_color_to_imu_rx} ${l515_cam_color_to_imu_ry} ${l515_cam_color_to_imu_rz}" />
-        <parent link="${name}_color_frame" />
-        <child link="${name}_gyro_frame" />
+        <parent link="${name}color_frame" />
+        <child link="${name}gyro_frame" />
       </joint>
-      <joint name="${name}_gyro_optical_joint" type="fixed">
+      <joint name="${name}gyro_optical_joint" type="fixed">
         <origin xyz = "0 0 0" rpy = "${-M_PI/2} 0 ${-M_PI/2}" />
-        <parent link="${name}_gyro_frame" />
-        <child link="${name}_gyro_optical_frame" />
+        <parent link="${name}gyro_frame" />
+        <child link="${name}gyro_optical_frame" />
       </joint>
-      <joint name="${name}_accel_joint" type="fixed">
+      <joint name="${name}accel_joint" type="fixed">
         <origin xyz = "${l515_cam_color_to_imu_px} ${l515_cam_color_to_imu_py} ${l515_cam_color_to_imu_pz}" rpy = "${l515_cam_color_to_imu_rx} ${l515_cam_color_to_imu_ry} ${l515_cam_color_to_imu_rz}" />
-        <parent link="${name}_color_frame" />
-        <child link="${name}_accel_frame" />
+        <parent link="${name}color_frame" />
+        <child link="${name}accel_frame" />
       </joint>
-      <joint name="${name}_accel_optical_joint" type="fixed">
+      <joint name="${name}accel_optical_joint" type="fixed">
         <origin xyz = "0 0 0" rpy = "${-M_PI/2} 0 ${-M_PI/2}" />
-        <parent link="${name}_accel_frame" />
-        <child link="${name}_accel_optical_frame" />
+        <parent link="${name}accel_frame" />
+        <child link="${name}accel_optical_frame" />
       </joint>
     </xacro:if>
     <xacro:if value="${add_plug}">
-      <xacro:usb_plug parent="${name}_bottom_screw_frame" name="${name}_usb_plug">
+      <xacro:usb_plug parent="${name}bottom_screw_frame" name="${name}usb_plug">
         <origin xyz="${l515_cam_mount_from_glass_offset-0.0148} -0.018 0.018" rpy="${M_PI/4} 0 0 "/>
       </xacro:usb_plug>

Commit message: updated tf names to not require camera name to hold _

File: realsense2_description/urdf/_l515.urdf.xacro (robot description, xacro)
@@ -46,16 +46,16 @@
     <xacro:property name="l515_cam_color_to_imu_rz" value="0.016301375"/>
     <!-- camera body, with origin at bottom screw mount -->
-    <joint name="${name}joint" type="fixed">
+    <joint name="${name}_joint" type="fixed">
       <xacro:insert_block name="origin" />
       <parent link="${parent}"/>
-      <child link="${name}bottom_screw_frame" />
+      <child link="${name}_bottom_screw_frame" />
     </joint>
-    <link name="${name}bottom_screw_frame"/>
-    <joint name="${name}link_joint" type="fixed">
+    <link name="${name}_bottom_screw_frame"/>
+    <joint name="${name}_link_joint" type="fixed">
       <origin xyz="${l515_cam_depth_px} ${l515_cam_depth_py} ${l515_cam_depth_pz}" rpy="0 0 0"/>
-      <parent link="${name}bottom_screw_frame"/>
-      <child link="${name}link" />
+      <parent link="${name}_bottom_screw_frame"/>
+      <child link="${name}_link" />
     </joint>
-    <link name="${name}link">
+    <link name="${name}_link">
       <visual>
         <!-- the mesh origin is in the middle of the front plate -->
@@ -88,85 +88,85 @@
       </inertial>
     </link>
-    <joint name="${name}lower_mount_joint" type="fixed">
+    <joint name="${name}_lower_mount_joint" type="fixed">
       <origin xyz="${l515_cam_mount_from_glass_offset-l515_cam_depth} 0 ${l515_cam_center-abs_mount_from_center}" rpy="0 0 0" />
-      <parent link="${name}bottom_screw_frame" />
-      <child link="${name}lower_mount" />
+      <parent link="${name}_bottom_screw_frame" />
+      <child link="${name}_lower_mount" />
     </joint>
-    <link name="${name}lower_mount"/>
-    <joint name="${name}upper_mount_joint" type="fixed">
+    <link name="${name}_lower_mount"/>
+    <joint name="${name}_upper_mount_joint" type="fixed">
       <origin xyz="${l515_cam_mount_from_glass_offset-l515_cam_depth} 0 ${l515_cam_center+abs_mount_from_center}" rpy="0 0 0" />
-      <parent link="${name}bottom_screw_frame" />
-      <child link="${name}upper_mount" />
+      <parent link="${name}_bottom_screw_frame" />
+      <child link="${name}_upper_mount" />
     </joint>
-    <link name="${name}upper_mount"/>
+    <link name="${name}_upper_mount"/>
     <!-- Use the nominal extrinsics between camera frames if the calibrated extrinsics aren't being published. e.g. running the device in simulation  -->
     <xacro:if value="${use_nominal_extrinsics}">
       <!-- camera depth joints and links -->
-      <joint name="${name}depth_joint" type="fixed">
+      <joint name="${name}_depth_joint" type="fixed">
         <origin xyz="0 0 0" rpy="0 0 0"/>
-        <parent link="${name}link"/>
-        <child link="${name}depth_frame" />
+        <parent link="${name}_link"/>
+        <child link="${name}_depth_frame" />
       </joint>
-      <link name="${name}depth_frame"/>
-      <joint name="${name}depth_optical_joint" type="fixed">
+      <link name="${name}_depth_frame"/>
+      <joint name="${name}_depth_optical_joint" type="fixed">
         <origin xyz="0 0 0" rpy="${-M_PI/2} 0 ${-M_PI/2}" />
-        <parent link="${name}depth_frame" />
-        <child link="${name}depth_optical_frame" />
+        <parent link="${name}_depth_frame" />
+        <child link="${name}_depth_optical_frame" />
       </joint>
-      <link name="${name}depth_optical_frame"/>
+      <link name="${name}_depth_optical_frame"/>
       <!-- camera left IR joints and links -->
-      <joint name="${name}infra_joint" type="fixed">
+      <joint name="${name}_infra_joint" type="fixed">
         <origin xyz="0 ${l515_cam_depth_to_infra_offset} 0" rpy="0 0 0" />
-        <parent link="${name}link" />
-        <child link="${name}infra_frame" />
+        <parent link="${name}_link" />
+        <child link="${name}_infra_frame" />
       </joint>
-      <link name="${name}infra_frame"/>
-      <joint name="${name}infra_optical_joint" type="fixed">
+      <link name="${name}_infra_frame"/>
+      <joint name="${name}_infra_optical_joint" type="fixed">
         <origin xyz="0 0 0" rpy="${-M_PI/2} 0 ${-M_PI/2}" />
-        <parent link="${name}infra_frame" />
-        <child link="${name}infra_optical_frame" />
+        <parent link="${name}_infra_frame" />
+        <child link="${name}_infra_optical_frame" />
       </joint>
-      <link name="${name}infra_optical_frame"/>
+      <link name="${name}_infra_optical_frame"/>
       <!-- camera color joints and links -->
-      <joint name="${name}color_joint" type="fixed">
+      <joint name="${name}_color_joint" type="fixed">
         <origin xyz="0 0 ${-l515_cam_transmitter_to_depth_pz+l515_cam_transmitter_to_color_pz}" rpy="0 0 0" />
-        <parent link="${name}link" />
-        <child link="${name}color_frame" />
+        <parent link="${name}_link" />
+        <child link="${name}_color_frame" />
       </joint>
-      <link name="${name}color_frame"/>
-      <joint name="${name}color_optical_joint" type="fixed">
+      <link name="${name}_color_frame"/>
+      <joint name="${name}_color_optical_joint" type="fixed">
         <origin xyz="0 0 0" rpy="${-M_PI/2} 0 ${-M_PI/2}" />
-        <parent link="${name}color_frame" />
-        <child link="${name}color_optical_frame" />
+        <parent link="${name}_color_frame" />
+        <child link="${name}_color_optical_frame" />
       </joint>
-      <link name="${name}color_optical_frame"/>
+      <link name="${name}_color_optical_frame"/>
       <!-- camera IMU joints and links -->
-      <link name="${name}gyro_frame" />
-      <link name="${name}gyro_optical_frame" />
-      <link name="${name}accel_frame" />
-      <link name="${name}accel_optical_frame" />
-      <joint name="${name}gyro_joint" type="fixed">
+      <link name="${name}_gyro_frame" />
+      <link name="${name}_gyro_optical_frame" />
+      <link name="${name}_accel_frame" />
+      <link name="${name}_accel_optical_frame" />
+      <joint name="${name}_gyro_joint" type="fixed">
         <origin xyz = "${l515_cam_color_to_imu_px} ${l515_cam_color_to_imu_py} ${l515_cam_color_to_imu_pz}" rpy = "${l515_cam_color_to_imu_rx} ${l515_cam_color_to_imu_ry} ${l515_cam_color_to_imu_rz}" />
-        <parent link="${name}color_frame" />
-        <child link="${name}gyro_frame" />
+        <parent link="${name}_color_frame" />
+        <child link="${name}_gyro_frame" />
       </joint>
-      <joint name="${name}gyro_optical_joint" type="fixed">
+      <joint name="${name}_gyro_optical_joint" type="fixed">
         <origin xyz = "0 0 0" rpy = "${-M_PI/2} 0 ${-M_PI/2}" />
-        <parent link="${name}gyro_frame" />
-        <child link="${name}gyro_optical_frame" />
+        <parent link="${name}_gyro_frame" />
+        <child link="${name}_gyro_optical_frame" />
       </joint>
-      <joint name="${name}accel_joint" type="fixed">
+      <joint name="${name}_accel_joint" type="fixed">
         <origin xyz = "${l515_cam_color_to_imu_px} ${l515_cam_color_to_imu_py} ${l515_cam_color_to_imu_pz}" rpy = "${l515_cam_color_to_imu_rx} ${l515_cam_color_to_imu_ry} ${l515_cam_color_to_imu_rz}" />
-        <parent link="${name}color_frame" />
-        <child link="${name}accel_frame" />
+        <parent link="${name}_color_frame" />
+        <child link="${name}_accel_frame" />
       </joint>
-      <joint name="${name}accel_optical_joint" type="fixed">
+      <joint name="${name}_accel_optical_joint" type="fixed">
         <origin xyz = "0 0 0" rpy = "${-M_PI/2} 0 ${-M_PI/2}" />
-        <parent link="${name}accel_frame" />
-        <child link="${name}accel_optical_frame" />
+        <parent link="${name}_accel_frame" />
+        <child link="${name}_accel_optical_frame" />
       </joint>
     </xacro:if>
     <xacro:if value="${add_plug}">
-      <xacro:usb_plug parent="${name}bottom_screw_frame" name="${name}usb_plug">
+      <xacro:usb_plug parent="${name}_bottom_screw_frame" name="${name}_usb_plug">
         <origin xyz="${l515_cam_mount_from_glass_offset-0.0148} -0.018 0.018" rpy="${M_PI/4} 0 0 "/>
       </xacro:usb_plug>
